File: Hardware/KiCad files/Mesh-IT.kicad_sch (KiCad schematic)
At the start: 17 parts, among them Q1 SS8050, U1 XIAO-ESP32-S3-DIP, U7 TCA8418RTWR

Commit message: Uploading final files
Changed lines of the file:
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@@
 	(text "I/o expander"
 		(exclude_from_sim no)
-		(at 248.666 44.958 0)
+		(at 237.236 68.072 0)
 		(effects
 			(font
@@
 	(text "GPS MODULE"
 		(exclude_from_sim no)
-		(at 168.656 34.29 0)
+		(at 169.164 36.576 0)
 		(effects
 			(font
@@
 			)
 		)
-	)
-	(rule_area
-		(exclude_from_sim no)
-		(in_bom yes)
-		(on_board yes)
-		(dnp no)
-		(polyline
-			(pts
-				(xy 55.88 76.2) (xy 93.345 75.565) (xy 94.615 76.835) (xy 95.25 114.3) (xy 55.88 114.3) (xy 55.88 76.2)
-			)
-			(stroke
-				(width 1.524)
-				(type solid)
-			)
-			(fill
-				(type none)
-			)
-		)
-	)
-	(rule_area
-		(exclude_from_sim no)
-		(in_bom yes)
-		(on_board yes)
-		(dnp no)
-		(polyline
-			(pts
-				(xy 207.01 38.1) (xy 207.01 38.1) (xy 207.01 81.28) (xy 207.01 81.28) (xy 146.05 81.28) (xy 146.05 76.2)
-				(xy 146.05 36.83) (xy 147.32 36.83)
-			)
-			(stroke
-				(width 1.524)
-				(type solid)
-			)
-			(fill
-				(type none)
-			)
-		)
-	)
-	(rule_area
-		(exclude_from_sim no)
-		(in_bom yes)
-		(on_board yes)
-		(dnp no)
-		(polyline
-			(pts
-				(xy 134.62 90.17) (xy 156.21 90.17) (xy 156.21 111.76) (xy 154.94 113.03) (xy 135.89 113.03) (xy 134.62 111.76)
-			)
-			(stroke
-				(width 1.524)
-				(type solid)
-			)
-			(fill
-				(type none)
-			)
-		)
-	)
-	(rule_area
-		(exclude_from_sim no)
-		(in_bom yes)
-		(on_board yes)
-		(dnp no)
-		(polyline
-			(pts
-				(xy 284.48 118.11) (xy 214.63 118.11) (xy 214.63 52.07) (xy 214.63 48.26) (xy 283.21 48.26) (xy 284.48 49.53)
-			)
-			(stroke
-				(width 1.524)
-				(type solid)
-			)
-			(fill
-				(type none)
-			)
-		)
-	)
-	(rule_area
-		(exclude_from_sim no)
-		(in_bom yes)
-		(on_board yes)
-		(dnp no)
-		(polyline
-			(pts
-				(xy 96.52 105.41) (xy 96.52 78.74) (xy 130.81 78.74) (xy 130.81 107.95) (xy 99.06 107.95)
-			)
-			(stroke
-				(width 1.524)
-				(type solid)
-			)
-			(fill
-				(type none)
-			)
-		)
-	)
-	(rule_area
-		(exclude_from_sim no)
-		(in_bom yes)
-		(on_board yes)
-		(dnp no)
-		(polyline
-			(pts
-				(xy 142.24 68.58) (xy 54.9275 69.215) (xy 54.2925 37.465) (xy 140.0174 37.465) (xy 140.97 38.1)
-			)
-			(stroke
-				(width 1.524)
-				(type solid)
-			)
-			(fill
-				(type none)
-			)
-		)
-	)
-	(rule_area
-		(exclude_from_sim no)
-		(in_bom yes)
-		(on_board yes)
-		(dnp no)
-		(polyline
-			(pts
-				(xy 83.82 123.19) (xy 154.94 123.19) (xy 154.94 194.31) (xy 81.28 194.31) (xy 78.74 191.77) (xy 78.74 128.27)
-			)
-			(stroke
-				(width 1.524)
-				(type solid)
-				(color 255 21 44 1)
-			)
-			(fill
-				(type none)
-			)
-		)
